File: BuckConverter/BuckConverter.kicad_pcb (KiCad board)
At the start: 2 copper layers, 8 parts, among them U1 LM358, U2 LAUNCHXL-F28379D

Commit message: Add all footprints
Parts:
- added C10: 10u, Capacitor_SMD:C_0805_2012Metric, F.Cu at (189.1, 67.5)
- added C11: 220n, Capacitor_SMD:C_0805_2012Metric, F.Cu at (189.1, 70.5)
- added C12: 10u, Capacitor_SMD:C_0805_2012Metric, F.Cu at (189.1, 73.5)
- added C3: 470u, Capacitor_THT:CP_Radial_D18.0mm_P7.50mm, F.Cu at (219.4, 20.4)
- added C4: 1u, Capacitor_SMD:C_0805_2012Metric_Pad1.18x1.45mm_HandSolder, F.Cu at (215.3, 57.2)
- added C5: ?, Capacitor_THT:CP_Radial_D18.0mm_P7.50mm, F.Cu at (219.4, 40.0)
- added C6: 1u, Capacitor_SMD:C_0805_2012Metric, F.Cu at (155.0, 84.5)
- added C7: 1u, Capacitor_SMD:C_0805_2012Metric, F.Cu at (155.0, 87.5)
- added C8: 1u, Capacitor_SMD:C_0805_2012Metric, F.Cu at (155.0, 90.5)
- added C9: C, Resistor_SMD:R_0805_2012Metric_Pad1.20x1.40mm_HandSolder, F.Cu at (150.4, 76.8)
- added D1: SS310, Diode_SMD:D_SMA, F.Cu at (228.5, 52.0)
- added D2: IR26-21C_L110_TR8, LED_SMD:LED_1206_3216Metric, F.Cu at (160.0, 89.2)
- added D3: IR26-21C_L110_TR8, LED_SMD:LED_1206_3216Metric, F.Cu at (173.6, 77.1)
- added D4: IR26-21C_L110_TR8, LED_SMD:LED_1206_3216Metric, F.Cu at (173.6, 80.5)
- added D5: US2AA, Diode_SMD:D_SMA, F.Cu at (161.2, 85.2)
- added D6: IR26-21C_L110_TR8, LED_SMD:LED_1206_3216Metric, F.Cu at (173.6, 83.8)
- added D7: IR26-21C_L110_TR8, LED_SMD:LED_1206_3216Metric, F.Cu at (160.0, 92.6)
- added J1: Conn_01x01_Pin, Connector:Banana_Jack_1Pin, F.Cu at (154.3, 16.9)
- added J2: Conn_01x01_Pin, Connector:Banana_Jack_1Pin, F.Cu at (154.3, 29.4)
- added J3: Conn_01x01_Pin, Connector:Banana_Jack_1Pin, F.Cu at (154.3, 42.0)
- added J4: Conn_01x01_Pin, Connector:Banana_Jack_1Pin, F.Cu at (154.3, 54.5)
- added J5: Conn_01x01_Pin, Connector:Banana_Jack_1Pin, F.Cu at (154.3, 67.1)
- added L1: ?, Inductor_THT:L_Radial_D50.8mm_P38.86mm_Vishay_IHB-6, F.Cu at (167.3, 36.8)
- added Q1: IRF540N, Package_TO_SOT_THT:TO-220-3_Vertical, F.Cu at (216.1, 53.6)
- added R10: R, Resistor_SMD:R_0805_2012Metric_Pad1.20x1.40mm_HandSolder, F.Cu at (150.4, 85.7)
- added R11: 7R, Resistor_SMD:R_0805_2012Metric_Pad1.20x1.40mm_HandSolder, F.Cu at (150.4, 88.7)
- added R12: 50R, Resistor_SMD:R_1206_3216Metric_Pad1.30x1.75mm_HandSolder, F.Cu at (165.8, 89.2)
- added R13: 3.3k, Resistor_SMD:R_0805_2012Metric_Pad1.20x1.40mm_HandSolder, F.Cu at (150.4, 91.6)
- added R5: 3.3k, Resistor_SMD:R_0805_2012Metric_Pad1.20x1.40mm_HandSolder, F.Cu at (150.4, 79.8)
- added R6: 3.3k, Resistor_SMD:R_0805_2012Metric_Pad1.20x1.40mm_HandSolder, F.Cu at (178.8, 76.8)
- added R7: 3.3k, Resistor_SMD:R_0805_2012Metric_Pad1.20x1.40mm_HandSolder, F.Cu at (178.8, 79.8)
- added R8: 12R, Resistor_SMD:R_0805_2012Metric_Pad1.20x1.40mm_HandSolder, F.Cu at (150.4, 82.8)
- added R9: 3.3k, Resistor_SMD:R_0805_2012Metric_Pad1.20x1.40mm_HandSolder, F.Cu at (178.8, 82.8)
- added U3: UCC5304DWVR, UCC5304DWVR:SOIC8_DWV_TEX, F.Cu at (159.8, 79.2)
- added U4: TMV 0512SHI, TMV_0512SHI:TMV-HI_SINGLE_TRP, F.Cu at (163.8, 67.5)
Connections:
- U2 pad J10_2: unconnected-(U2I-GND_J10-PadJ10_2) -> GND
- U2 pad J10_3: unconnected-(U2I-GND_J10__1-PadJ10_3) -> GND
- U2 pad J12_3: unconnected-(U2J-GND_J12-PadJ12_3) -> GND
- U2 pad J14_5: unconnected-(U2K-GND_J14-PadJ14_5) -> GND
- U2 pad J15_5: unconnected-(U2L-GND_J15-PadJ15_5) -> GND
- U2 pad J16_2: unconnected-(U2N-GND_J16-PadJ16_2) -> GND
- U2 pad J16_3: unconnected-(U2N-GND_J16__1-PadJ16_3) -> GND
- U2 pad J1_1: unconnected-(U2A-3.3V_J1-PadJ1_1) -> +3.3V
- U2 pad J21_2: unconnected-(U2M-TP21/GND-PadJ21_2) -> GND
- U2 pad J21_4: unconnected-(U2M-TP22/GND-PadJ21_4) -> GND
- U2 pad J21_6: unconnected-(U2M-TP23/GND-PadJ21_6) -> GND
- U2 pad J21_8: unconnected-(U2M-TP24/GND-PadJ21_8) -> GND
- U2 pad J2_10: unconnected-(U2B-GND_J2-PadJ2_10) -> GND
- U2 pad J3_2: unconnected-(U2C-GND_J3-PadJ3_2) -> GND
- U2 pad J3_3: unconnected-(U2C-ADCIN14/ANALOGIN-PadJ3_3) -> /VFILT
- U2 pad J6_10: unconnected-(U2F-GND_J6-PadJ6_10) -> GND
- U2 pad J7_1: unconnected-(U2G-+5V_J7-PadJ7_1) -> +5V
- U2 pad J7_2: unconnected-(U2G-GND_J7-PadJ7_2) -> GND
- U2 pad J8_5: unconnected-(U2H-GPIO11/PWMOUT6B-PadJ8_5) -> /PWM

Commit message: PCB Completed
Parts:
- C8: footprint Capacitor_SMD:C_0805_2012Metric -> Capacitor_SMD:C_0805_2012Metric_Pad1.18x1.45mm_HandSolder
- moved C3 171.8 mm to (71.5, 107.7)
- moved D1 154.2 mm to (80.1, 94.0), turned to -90 degrees
- moved Q1 151.9 mm to (69.2, 91.9)
- moved R8 150.1 mm to (29.8, 100.8)
- moved C4 147.7 mm to (72.7, 95.7)
- moved D5 144.9 mm to (30.0, 103.4)
- moved C10 143.6 mm to (49.6, 101.6)
- moved C11 143.4 mm to (49.6, 103.9)
- moved C12 143.2 mm to (49.6, 106.2)
- moved U4 136.7 mm to (33.8, 109.9)
- moved J1 126.7 mm to (32.7, 52.5)
- moved R6 124.6 mm to (59.8, 113.5)
- moved C6 123.8 mm to (33.1, 106.4)
- moved J4 123.7 mm to (32.7, 77.5)
- moved R9 121.1 mm to (29.8, 96.8)
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- renumbered D6 to D5, D5 to D6, R11 to R10, R8 to R11, R4 to R3, R3 to R4, R9 to R8, R10 to R9
Connections:
- net Net-(U3-IN) renamed /GD/PWM_FILT
- C1 pad 1: Net-(U1A--) -> Net-(U1A-+)
- C10 pad 2: /GD/ISO_GND -> /VSW
- C11 pad 2: /GD/ISO_GND -> /VSW
- C12 pad 2: /GD/ISO_GND -> /VSW
- C3 pad 1: Net-(Q1-D) -> /PowerStage/VIN
- C3 pad 2: Net-(D1-A) -> GND
- C4 pad 1: Net-(Q1-D) -> /PowerStage/VIN
- C4 pad 2: Net-(D1-A) -> GND
- C5 pad 1: Net-(C5-Pad1) -> /VOUT
- C5 pad 2: Net-(D1-A) -> GND
- C7 pad 2: /GD/ISO_GND -> /VSW
- D1 pad 1: Net-(D1-K) -> /VSW
- D1 pad 2: Net-(D1-A) -> GND
- D6 pad 1: Net-(D5-K) (its old number) -> Net-(D6-K)
- J3 pad 1: /PowerStage/Vout -> /VOUT
- L1 pad 1: Net-(D1-K) -> /VSW
- L1 pad 2: Net-(C5-Pad1) -> /VOUT
- Q1 pad 2: Net-(Q1-D) -> /PowerStage/VIN
- Q1 pad 3: Net-(D1-K) -> /VSW
- R1 pad 1: Net-(U1A-+) -> GND
- R1 pad 2: unconnected-(R1-Pad2) -> Net-(U1A--)
- R10 pad 2: Net-(D5-K) (its old number) -> /VG
- R11 pad 2: Net-(D5-K) (its old number) -> Net-(D6-K)
- R12 pad 1: unconnected-(R12-Pad1) -> /VG
- R12 pad 2: /VG -> /VSW
- R13 pad 2: /GD/ISO_GND -> /VSW
- R2 pad 1: Net-(R2-Pad1) -> Net-(U1A--)
- R2 pad 2: Net-(U1A-+) -> /LPF/VFLIT
- R3 pad 1: Net-(U1A--) -> Net-(U1A-+)
- R4 pad 1: Net-(U1A--) -> Net-(U1A-+)
- R4 pad 2: unconnected-(R3-Pad2) -> /VOUT
- R5 pad 2: /GD/ISO_GND -> /VSW
- U1 pad 1: Net-(R2-Pad1) -> /LPF/VFLIT
- U1 pad 8: unconnected-(U1C-V+-Pad8) -> +3.3V
- U3 pad 3: unconnected-(U3-VCCI-Pad3) -> +5V
- U3 pad 5: /GD/ISO_GND -> /VSW
- U3 pad 6: /GD/ISO_GND -> /VSW
- U4 pad 5: /GD/ISO_GND -> /VSW
Routing:
- net /VSW: track 0.00 -> 136.3 mm, vias 0 -> 1
- net /PWM: track 0.00 -> 86.9 mm
- net +5V: track 0.00 -> 80.6 mm
- net /VOUT: track 0.00 -> 77.9 mm
- net /PowerStage/VIN: track 0.00 -> 76.7 mm
- net +3.3V: track 0.00 -> 36.9 mm
- net /GD/ISO_12: track 0.00 -> 26.4 mm
- net /VG: track 0.00 -> 21.1 mm
- net /GD/PWM_FILT: track 0.00 -> 9.15 mm
- net /GD/GD_PWM: track 0.00 -> 7.78 mm
- net Net-(U1A-+): track 0.00 -> 7.69 mm
- net Net-(U1A--): track 0.00 -> 4.83 mm
- net Net-(D6-K): track 0.00 -> 3.96 mm
- net Net-(D5-K): track 0.00 -> 2.60 mm
- net Net-(D3-K): track 0.00 -> 2.58 mm
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- added copper zone on B.Cu, net GND
- added copper zone on F.Cu, net GND
Other:
- board outline added: 130.3 x 135.9 mm
- board text added: "+3V"
- board text added: "+5V"
- board text added: "GD PWM"
- board text added: "ISO 12"
- board text added: "PWM"
