File: BuckConverter/MCU.kicad_sch (KiCad schematic)
At the start: 7 parts, among them U2 LAUNCHXL-F28379D

Commit message: PCB Completed
Parts:
- renumbered D6 to D5, R9 to R8
Connections:
- no-connect marks 90 -> 89
Changed lines of the file:
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@@
 	)
 	(no_connect
-		(at 161.29 69.85)
-	)
-	(no_connect
 		(at 160.02 36.83)
 	)
@@
 		(on_board yes)
 		(dnp no)
-		(property "Reference" "D6"
+		(property "Reference" "D5"
 			(at 84.074 36.576 90)
 			(effects
@@
 			(project "BuckConverter"
 				(path "/fd6bac42-b74a-4329-b064-b676c79abc2c/b0f193ef-9a87-4c47-af17-4207c54df54c"
-					(reference "D6")
+					(reference "D5")
 					(unit 1)
 				)
@@
 		(on_board yes)
 		(dnp no)
-		(property "Reference" "R9"
+		(property "Reference" "R8"
 			(at 95.2499 36.83 0)
 			(effects
@@
 			(project "BuckConverter"
 				(path "/fd6bac42-b74a-4329-b064-b676c79abc2c/b0f193ef-9a87-4c47-af17-4207c54df54c"
-					(reference "R9")
+					(reference "R8")
 					(unit 1)
 				)

Commit message: updated BOM
Parts:
- D3, D4, D5: Part Number (none) -> IR26-21C_L110_TR8
- U2: Part Number (none) -> LAUNCHXL-F28379D
Changed lines of the file:
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@@
 			)
 		)
-		(property "Part Number" ""
+		(property "Part Number" "LAUNCHXL-F28379D"
 			(at 45.72 167.64 0)
 			(effects
@@
 			)
 		)
-		(property "Part Number" ""
+		(property "Part Number" "LAUNCHXL-F28379D"
 			(at 228.6 44.45 0)
 			(effects
@@
 			)
 		)
-		(property "Part Number" ""
+		(property "Part Number" "LAUNCHXL-F28379D"
 			(at 40.64 67.31 0)
 			(effects
@@
 			)
 		)
-		(property "Part Number" ""
+		(property "Part Number" "LAUNCHXL-F28379D"
 			(at 214.63 146.05 0)
 			(effects
@@
 			)
 		)
+		(property "Part Number" "IR26-21C_L110_TR8"
+			(at 85.09 20.32 0)
+			(effects
+				(font
+					(size 1.27 1.27)
+				)
+				(hide yes)
+			)
+		)
 		(pin "1"
 		)
@@
 			)
 		)
-		(property "Part Number" ""
+		(property "Part Number" "LAUNCHXL-F28379D"
 			(at 199.39 134.62 0)
 			(effects
@@
 			)
 		)
-		(property "Part Number" ""
+		(property "Part Number" "LAUNCHXL-F28379D"
 			(at 224.79 69.85 0)
 			(effects
@@
 			)
 		)
-		(property "Part Number" ""
+		(property "Part Number" "LAUNCHXL-F28379D"
 			(at 181.61 77.47 0)
 			(effects
@@
 			)
 		)
-		(property "Part Number" ""
+		(property "Part Number" "LAUNCHXL-F28379D"
 			(at 41.91 100.33 0)
 			(effects
@@
 			)
 		)
-		(property "Part Number" ""
+		(property "Part Number" "LAUNCHXL-F28379D"
 			(at 180.34 39.37 0)
 			(effects
@@
 			)
 		)
+		(property "Part Number" "IR26-21C_L110_TR8"
+			(at 83.82 39.37 0)
+			(effects
+				(font
+					(size 1.27 1.27)
+				)
+				(hide yes)
+			)
+		)
 		(pin "1"
 		)
@@
 			)
 		)
+		(property "Part Number" "IR26-21C_L110_TR8"
+			(at 85.09 30.48 0)
+			(effects
+				(font
+					(size 1.27 1.27)
+				)
+				(hide yes)
+			)
+		)
 		(pin "1"
 		)
@@
 			)
 		)
-		(property "Part Number" ""
+		(property "Part Number" "LAUNCHXL-F28379D"
 			(at 219.71 97.79 0)
 			(effects
@@
 			)
 		)
-		(property "Part Number" ""
+		(property "Part Number" "LAUNCHXL-F28379D"
 			(at 180.34 109.22 0)
 			(effects
@@
 			)
 		)
-		(property "Part Number" ""
+		(property "Part Number" "LAUNCHXL-F28379D"
 			(at 223.52 118.11 0)
 			(effects
@@
 			)
 		)
-		(property "Part Number" ""
+		(property "Part Number" "LAUNCHXL-F28379D"
 			(at 246.38 133.35 0)
 			(effects
@@
 			)
 		)
-		(property "Part Number" ""
+		(property "Part Number" "LAUNCHXL-F28379D"
 			(at 44.45 134.62 0)
 			(effects
