File: BuckConverter/MCU.kicad_sch (KiCad schematic)
At the start: 7 parts, among them U2 LAUNCHXL-F28379D

Commit message: Update PCB and BOM
Changed lines of the file:
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@@
 	(wire
 		(pts
-			(xy 79.375 39.37) (xy 80.01 39.37)
+			(xy 78.74 39.37) (xy 80.01 39.37)
 		)
 		(stroke
@@
 	)
 	(label "PWM"
-		(at 79.375 39.37 180)
+		(at 78.74 39.37 180)
 		(effects
 			(font
