File: BuckConverter/GD.kicad_sch (KiCad schematic)
At the start: 18 parts, among them U3 UCC5304DWVR, U4 TMV 0512SHI

Commit message: Add all footprints
Parts:
- removed U3: UCC5304DWVR, SOIC8_DWV_TEX, symbol 2025-02-01_23-04-27:UCC5304DWVR
- added U3: UCC5304DWVR, SOIC8_DWV_TEX, symbol 2025-02-16_19-57-41:UCC5304DWVR
- C10, C11, C12: footprint (none) -> Capacitor_SMD:C_0805_2012Metric
Connections:
- net +5V: now also U3.2 (VCCI)
- net GD_PWM: now also U3.7 (OUT)
- net GND: now also U3.4 (GND)
- net ISO_12: now also U3.8 (VDD)
- net ISO_GND: now also U3.5 (VSS), U3.6 (VSS)
- net at C9.1, R10.2: now also U3.1 (IN)
Changed lines of the file:
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@@
 			)
 		)
-		(property "Footprint" ""
+		(property "Footprint" "Capacitor_SMD:C_0805_2012Metric"
 			(at 135.5852 118.11 0)
 			(effects
@@
 			)
 		)
-		(property "Description" "Bypass Capcitor"
+		(property "Description" "Unpolarized capacitor"
 			(at 134.62 114.3 0)
 			(effects
@@
 			)
 		)
-		(property "Footprint" ""
+		(property "Footprint" "Capacitor_SMD:C_0805_2012Metric"
 			(at 154.6352 118.11 0)
 			(effects
@@
 	)
 	(symbol
-		(lib_id "2025-02-01_23-04-27:UCC5304DWVR")
+		(lib_id "power:+5V")
+		(at 81.28 48.26 0)
+		(unit 1)
+		(exclude_from_sim no)
+		(in_bom yes)
+		(on_board yes)
+		(dnp no)
+		(fields_autoplaced yes)
+		(property "Reference" "#PWR042"
+			(at 81.28 52.07 0)
+			(effects
+				(font
+					(size 1.27 1.27)
+				)
+				(hide yes)
+			)
+		)
+		(property "Value" "+5V"
+			(at 81.28 43.18 0)
+			(effects
+				(font
+					(size 1.27 1.27)
+				)
+			)
+		)
+		(property "Footprint" ""
+			(at 81.28 48.26 0)
+			(effects
+				(font
+					(size 1.27 1.27)
+				)
+				(hide yes)
+			)
+		)
+		(property "Datasheet" ""
+			(at 81.28 48.26 0)
+			(effects
+				(font
+					(size 1.27 1.27)
+				)
+				(hide yes)
+			)
+		)
+		(property "Description" "Power symbol creates a global label with name \"+5V\""
+			(at 81.28 48.26 0)
+			(effects
+				(font
+					(size 1.27 1.27)
+				)
+				(hide yes)
+			)
+		)
+		(pin "1"
+		)
+		(instances
+			(project ""
+				(path "/fd6bac42-b74a-4329-b064-b676c79abc2c/4500e0af-ac1d-424f-9007-f4139dc7a85a"
+					(reference "#PWR042")
+					(unit 1)
+				)
+			)
+		)
+	)
+	(symbol
+		(lib_id "power:GND")
+		(at 24.13 31.75 90)
+		(unit 1)
+		(exclude_from_sim no)
+		(in_bom yes)
+		(on_board yes)
+		(dnp no)
+		(fields_autoplaced yes)
+		(property "Reference" "#PWR041"
+			(at 30.48 31.75 0)
+			(effects
+				(font
+					(size 1.27 1.27)
+				)
+				(hide yes)
+			)
+		)
+		(property "Value" "GND"
+			(at 27.94 31.7499 90)
+			(effects
+				(font
+					(size 1.27 1.27)
+				)
+				(justify right)
+			)
+		)
+		(property "Footprint" ""
+			(at 24.13 31.75 0)
+			(effects
+				(font
+					(size 1.27 1.27)
+				)
+				(hide yes)
+			)
+		)
+		(property "Datasheet" ""
+			(at 24.13 31.75 0)
+			(effects
+				(font
+					(size 1.27 1.27)
+				)
+				(hide yes)
+			)
+		)
+		(property "Description" "Power symbol creates a global label with name \"GND\" , ground"
+			(at 24.13 31.75 0)
+			(effects
+				(font
+					(size 1.27 1.27)
+				)
+				(hide yes)
+			)
+		)
+		(pin "1"
+		)
+		(instances
+			(project ""
+				(path "/fd6bac42-b74a-4329-b064-b676c79abc2c/4500e0af-ac1d-424f-9007-f4139dc7a85a"
+					(reference "#PWR041")
+					(unit 1)
+				)
+			)
+		)
+	)
+	(symbol
+		(lib_id "power:GND")
+		(at 100.33 87.63 270)
+		(unit 1)
+		(exclude_from_sim no)
+		(in_bom yes)
+		(on_board yes)
+		(dnp no)
+		(fields_autoplaced yes)
+		(property "Reference" "#PWR052"
+			(at 93.98 87.63 0)
+			(effects
+				(font
+					(size 1.27 1.27)
+				)
+				(hide yes)
+			)
+		)
+		(property "Value" "GND"
+			(at 96.52 87.6299 90)
+			(effects
+				(font
+					(size 1.27 1.27)
+				)
+				(justify right)
+			)
+		)
+		(property "Footprint" ""
+			(at 100.33 87.63 0)
+			(effects
+				(font
+					(size 1.27 1.27)
+				)
+				(hide yes)
+			)
+		)
+		(property "Datasheet" ""
+			(at 100.33 87.63 0)
+			(effects
+				(font
+					(size 1.27 1.27)
+				)
+				(hide yes)
+			)
+		)
+		(property "Description" "Power symbol creates a global label with name \"GND\" , ground"
+			(at 100.33 87.63 0)
+			(effects
+				(font
+					(size 1.27 1.27)
+				)
+				(hide yes)
+			)
+		)
+		(pin "1"
+		)
+		(instances
+			(project "BuckConverter"
+				(path "/fd6bac42-b74a-4329-b064-b676c79abc2c/4500e0af-ac1d-424f-9007-f4139dc7a85a"
+					(reference "#PWR052")
+					(unit 1)
+				)
+			)
+		)
+	)
+	(symbol
+		(lib_id "2025-02-16_19-57-41:UCC5304DWVR")
 		(at 100.33 80.01 0)
 		(unit 1)
@@
 			)
 		)
+		(pin "8"
+		)
+		(pin "2"
+		)
+		(pin "5"
+		)
+		(pin "3"
+		)
+		(pin "7"
+		)
 		(pin "6"
 		)
-		(pin "8"
-		)
-		(pin "2"
-		)
-		(pin "5"
+		(pin "1"
 		)
 		(pin "4"
 		)
-		(pin "3"
-		)
-		(pin "7"
-		)
-		(pin "1"
-		)
 		(instances
 			(project ""
 				(path "/fd6bac42-b74a-4329-b064-b676c79abc2c/4500e0af-ac1d-424f-9007-f4139dc7a85a"
 					(reference "U3")
-					(unit 1)
-				)
-			)
-		)
-	)
-	(symbol
-		(lib_id "power:+5V")
-		(at 81.28 48.26 0)
-		(unit 1)
-		(exclude_from_sim no)
-		(in_bom yes)
-		(on_board yes)
-		(dnp no)
-		(fields_autoplaced yes)
-		(property "Reference" "#PWR042"
-			(at 81.28 52.07 0)
-			(effects
-				(font
-					(size 1.27 1.27)
-				)
-				(hide yes)
-			)
-		)
-		(property "Value" "+5V"
-			(at 81.28 43.18 0)
-			(effects
-				(font
-					(size 1.27 1.27)
-				)
-			)
-		)
-		(property "Footprint" ""
-			(at 81.28 48.26 0)
-			(effects
-				(font
-					(size 1.27 1.27)
-				)
-				(hide yes)
-			)
-		)
-		(property "Datasheet" ""
-			(at 81.28 48.26 0)
-			(effects
-				(font
-					(size 1.27 1.27)
-				)
-				(hide yes)
-			)
-		)
-		(property "Description" "Power symbol creates a global label with name \"+5V\""
-			(at 81.28 48.26 0)
-			(effects
-				(font
-					(size 1.27 1.27)
-				)
-				(hide yes)
-			)
-		)
-		(pin "1"
-		)
-		(instances
-			(project ""
-				(path "/fd6bac42-b74a-4329-b064-b676c79abc2c/4500e0af-ac1d-424f-9007-f4139dc7a85a"
-					(reference "#PWR042")
-					(unit 1)
-				)
-			)
-		)
-	)
-	(symbol
-		(lib_id "power:GND")
-		(at 24.13 31.75 90)
-		(unit 1)
-		(exclude_from_sim no)
-		(in_bom yes)
-		(on_board yes)
-		(dnp no)
-		(fields_autoplaced yes)
-		(property "Reference" "#PWR041"
-			(at 30.48 31.75 0)
-			(effects
-				(font
-					(size 1.27 1.27)
-				)
-				(hide yes)
-			)
-		)
-		(property "Value" "GND"
-			(at 27.94 31.7499 90)
-			(effects
-				(font
-					(size 1.27 1.27)
-				)
-				(justify right)
-			)
-		)
-		(property "Footprint" ""
-			(at 24.13 31.75 0)
-			(effects
-				(font
-					(size 1.27 1.27)
-				)
-				(hide yes)
-			)
-		)
-		(property "Datasheet" ""
-			(at 24.13 31.75 0)
-			(effects
-				(font
-					(size 1.27 1.27)
-				)
-				(hide yes)
-			)
-		)
-		(property "Description" "Power symbol creates a global label with name \"GND\" , ground"
-			(at 24.13 31.75 0)
-			(effects
-				(font
-					(size 1.27 1.27)
-				)
-				(hide yes)
-			)
-		)
-		(pin "1"
-		)
-		(instances
-			(project ""
-				(path "/fd6bac42-b74a-4329-b064-b676c79abc2c/4500e0af-ac1d-424f-9007-f4139dc7a85a"
-					(reference "#PWR041")
-					(unit 1)
-				)
-			)
-		)
-	)
-	(symbol
-		(lib_id "power:GND")
-		(at 100.33 87.63 270)
-		(unit 1)
-		(exclude_from_sim no)
-		(in_bom yes)
-		(on_board yes)
-		(dnp no)
-		(fields_autoplaced yes)
-		(property "Reference" "#PWR052"
-			(at 93.98 87.63 0)
-			(effects
-				(font
-					(size 1.27 1.27)
-				)
-				(hide yes)
-			)
-		)
-		(property "Value" "GND"
-			(at 96.52 87.6299 90)
-			(effects
-				(font
-					(size 1.27 1.27)
-				)
-				(justify right)
-			)
-		)
-		(property "Footprint" ""
-			(at 100.33 87.63 0)
-			(effects
-				(font
-					(size 1.27 1.27)
-				)
-				(hide yes)
-			)
-		)
-		(property "Datasheet" ""
-			(at 100.33 87.63 0)
-			(effects
-				(font
-					(size 1.27 1.27)
-				)
-				(hide yes)
-			)
-		)
-		(property "Description" "Power symbol creates a global label with name \"GND\" , ground"
-			(at 100.33 87.63 0)
-			(effects
-				(font
-					(size 1.27 1.27)
-				)
-				(hide yes)
-			)
-		)
-		(pin "1"
-		)
-		(instances
-			(project "BuckConverter"
-				(path "/fd6bac42-b74a-4329-b064-b676c79abc2c/4500e0af-ac1d-424f-9007-f4139dc7a85a"
-					(reference "#PWR052")
 					(unit 1)
 				)
@@
 			)
 		)
-		(property "Footprint" ""
+		(property "Footprint" "Capacitor_SMD:C_0805_2012Metric"
 			(at 169.8752 118.11 0)
 			(effects

Commit message: PCB Completed
Parts:
- C8: footprint Capacitor_SMD:C_0805_2012Metric -> Capacitor_SMD:C_0805_2012Metric_Pad1.18x1.45mm_HandSolder
- renumbered D5 to D6, R11 to R10, R8 to R11, R10 to R9
Connections:
- net ISO_GND is gone; now on net VSW: C10.2, C11.2, C12.2, C7.2, R13.2, R5.2, U3.5 (VSS), U3.6 (VSS), U4.5 (-VOUT)
- net +5V: now also U3.3 (VCCI)
- net VG: now also R10.2, R12.1; no longer R12.2
- net VSW: now also R12.2
- net at D6.1 (K), R11.2: no longer R10.2
- net PWM_FILT: now reaches C9.1, R9.2, U3.1 (IN)
Other:
- moved on the sheet: R12, R9
Changed lines of the file:
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@@
+	)
+	(junction
+		(at 100.33 82.55)
+		(diameter 0)
+		(color 0 0 0 0)
 	)
 	(junction
@@
 	)
 	(junction
-		(at 177.8 82.55)
+		(at 191.77 90.17)
 		(diameter 0)
 		(color 0 0 0 0)
@@
 	(wire
 		(pts
-			(xy 177.8 90.17) (xy 177.8 82.55)
-		)
-		(stroke
-			(width 0)
-			(type default)
-		)
-	)
-	(wire
-		(pts
 			(xy 165.1 82.55) (xy 167.64 82.55)
 		)
@@
 	(wire
 		(pts
-			(xy 177.8 82.55) (xy 179.07 82.55)
-		)
-		(stroke
-			(width 0)
-			(type default)
-		)
-	)
-	(wire
-		(pts
 			(xy 189.23 46.99) (xy 189.23 50.8)
 		)
@@
 	(wire
 		(pts
+			(xy 100.33 82.55) (xy 100.33 85.09)
+		)
+		(stroke
+			(width 0)
+			(type default)
+		)
+	)
+	(wire
+		(pts
 			(xy 81.28 63.5) (xy 81.28 67.31)
 		)
@@
 	(wire
 		(pts
-			(xy 175.26 90.17) (xy 177.8 90.17)
+			(xy 191.77 100.33) (xy 191.77 99.06)
+		)
+		(stroke
+			(width 0)
+			(type default)
+		)
+	)
+	(wire
+		(pts
+			(xy 175.26 90.17) (xy 191.77 90.17)
 		)
 		(stroke
@@
 	(wire
 		(pts
-			(xy 78.74 78.74) (xy 82.55 78.74)
+			(xy 78.74 80.01) (xy 82.55 80.01)
 		)
 		(stroke
@@
 	(wire
 		(pts
-			(xy 175.26 82.55) (xy 177.8 82.55)
+			(xy 175.26 82.55) (xy 179.07 82.55)
 		)
 		(stroke
@@
 	(wire
 		(pts
-			(xy 82.55 78.74) (xy 82.55 80.01)
-		)
-		(stroke
-			(width 0)
-			(type default)
-		)
-	)
-	(wire
-		(pts
 			(xy 81.28 52.07) (xy 81.28 55.88)
 		)
@@
 	(wire
 		(pts
-			(xy 191.77 91.44) (xy 191.77 82.55)
+			(xy 191.77 91.44) (xy 191.77 90.17)
 		)
 		(stroke
@@
 		(pts
 			(xy 152.4 60.96) (xy 163.83 60.96)
+		)
+		(stroke
+			(width 0)
+			(type default)
+		)
+	)
+	(wire
+		(pts
+			(xy 191.77 90.17) (xy 191.77 82.55)
+		)
+		(stroke
+			(width 0)
+			(type default)
+		)
+	)
+	(wire
+		(pts
+			(xy 69.85 80.01) (xy 71.12 80.01)
 		)
 		(stroke
@@
 		)
 	)
+	(label "ISO_GND"
+		(at 191.77 100.33 270)
+		(effects
+			(font
+				(size 1.27 1.27)
+			)
+			(justify right bottom)
+		)
+	)
+	(label "PWM_FILT"
+		(at 82.55 80.01 0)
+		(effects
+			(font
+				(size 1.27 1.27)
+			)
+			(justify left bottom)
+		)
+	)
 	(label "VG"
 		(at 215.9 92.71 0)
@@
 		)
 	)
+	(label "ISO_GND"
+		(at 55.88 25.4 180)
+		(effects
+			(font
+				(size 1.27 1.27)
+			)
+			(justify right bottom)
+		)
+	)
 	(label "ISO_12"
 		(at 140.97 80.01 0)
@@
 	)
 	(label "PWM"
-		(at 71.12 78.74 180)
+		(at 69.85 80.01 180)
 		(effects
 			(font
@@
 			)
 			(justify left bottom)
-		)
-	)
-	(label "VSW"
-		(at 55.88 25.4 180)
-		(effects
-			(font
-				(size 1.27 1.27)
-			)
-			(justify right bottom)
 		)
 	)
@@
 			)
 		)
-		(property "Footprint" "Capacitor_SMD:C_0805_2012Metric"
+		(property "Footprint" "Capacitor_SMD:C_0805_2012Metric_Pad1.18x1.45mm_HandSolder"
 			(at 112.7252 110.49 0)
 			(effects
@@
 		(on_board yes)
 		(dnp no)
-		(property "Reference" "R8"
+		(property "Reference" "R11"
 			(at 171.45 78.232 90)
 			(effects
@@
 			(project "BuckConverter"
 				(path "/fd6bac42-b74a-4329-b064-b676c79abc2c/4500e0af-ac1d-424f-9007-f4139dc7a85a"
-					(reference "R8")
+					(reference "R11")
 					(unit 1)
 				)
@@
 		(on_board yes)
 		(dnp no)
-		(property "Reference" "R11"
+		(property "Reference" "R10"
 			(at 171.704 85.852 90)
 			(effects
@@
 			(project "BuckConverter"
 				(path "/fd6bac42-b74a-4329-b064-b676c79abc2c/4500e0af-ac1d-424f-9007-f4139dc7a85a"
-					(reference "R11")
+					(reference "R10")
 					(unit 1)
 				)
@@
 		(dnp no)
 		(fields_autoplaced yes)
-		(property "Reference" "D5"
+		(property "Reference" "D6"
 			(at 182.88 76.2 0)
 			(effects
@@
 			(project ""
 				(path "/fd6bac42-b74a-4329-b064-b676c79abc2c/4500e0af-ac1d-424f-9007-f4139dc7a85a"
-					(reference "D5")
+					(reference "D6")
 					(unit 1)
 				)
@@
 	(symbol
 		(lib_id "Device:R")
-		(at 191.77 95.25 180)
+		(at 191.77 95.25 0)
 		(unit 1)
 		(exclude_from_sim no)
@@
 					(size 1.27 1.27)
 				)
-				(justify right)
+				(justify left)
 			)
 		)
@@
 					(size 1.27 1.27)
 				)
-				(justify right)
+				(justify left)
 			)
 		)
 		(property "Footprint" "Resistor_SMD:R_1206_3216Metric_Pad1.30x1.75mm_HandSolder"
-			(at 193.548 95.25 90)
+			(at 189.992 95.25 90)
 			(effects
 				(font
@@
 	(symbol
 		(lib_id "Device:R")
-		(at 74.93 78.74 90)
+		(at 74.93 80.01 90)
 		(unit 1)
 		(exclude_from_sim no)
@@
 		(dnp no)
 		(fields_autoplaced yes)
-		(property "Reference" "R10"
-			(at 74.93 72.39 90)
+		(property "Reference" "R9"
+			(at 74.93 73.66 90)
 			(effects
 				(font
@@
 		)
 		(property "Value" "R"
-			(at 74.93 74.93 90)
+			(at 74.93 76.2 90)
 			(effects
 				(font
@@
 		)
 		(property "Footprint" "Resistor_SMD:R_0805_2012Metric_Pad1.20x1.40mm_HandSolder"
-			(at 74.93 80.518 90)
+			(at 74.93 81.788 90)
 			(effects
 				(font
@@
 		)
 		(property "Datasheet" "~"
-			(at 74.93 78.74 0)
+			(at 74.93 80.01 0)
 			(effects
 				(font
@@
 		)
 		(property "Description" "Resistor"
-			(at 74.93 78.74 0)
+			(at 74.93 80.01 0)
 			(effects
 				(font
@@
 		)
 		(property "Part Number" ""
-			(at 74.93 78.74 0)
+			(at 74.93 80.01 0)
 			(effects
 				(font
@@
 			(project ""
 				(path "/fd6bac42-b74a-4329-b064-b676c79abc2c/4500e0af-ac1d-424f-9007-f4139dc7a85a"
-					(reference "R10")
-					(unit 1)
-				)
+					(reference "R9")
+					(unit 1)
+				)

Commit message: PCB Final Draft
Parts:
- removed C9: C, Resistor_SMD:R_0805_2012Metric_Pad1.20x1.40mm_HandSolder, symbol Device:C
- removed R9: R, Resistor_SMD:R_0805_2012Metric_Pad1.20x1.40mm_HandSolder, symbol Device:R
- added C9: 33p, CAP_600F0R1AT250T_ATC, symbol 600F330FT250XT4K:600F330FT250XT
- added R9: 51, RC0805N_YAG, symbol RC0805FR_0751RL:RC0805FR-0751RL
Connections:
- net GND: now also C9.2
- net PWM: now also R9.1
- net PWM_FILT: now also C9.1, R9.2
Changed lines of the file:
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@@
+	(wire
+		(pts
+			(xy 53.34 80.01) (xy 58.42 80.01)
+		)
+		(stroke
+			(width 0)
+			(type default)
+		)
+	)
 	(wire
 		(pts
@@
 	(wire
 		(pts
-			(xy 78.74 80.01) (xy 82.55 80.01)
+			(xy 71.12 80.01) (xy 82.55 80.01)
 		)
 		(stroke
@@
 		(pts
 			(xy 191.77 90.17) (xy 191.77 82.55)
-		)
-		(stroke
-			(width 0)
-			(type default)
-		)
-	)
-	(wire
-		(pts
-			(xy 69.85 80.01) (xy 71.12 80.01)
 		)
 		(stroke
@@
 	)
 	(label "PWM"
-		(at 69.85 80.01 180)
+		(at 53.34 80.01 180)
 		(effects
 			(font
@@
 	)
 	(symbol
+		(lib_id "600F330FT250XT4K:600F330FT250XT")
+		(at 82.55 82.55 270)
+		(unit 1)
+		(exclude_from_sim no)
+		(in_bom yes)
+		(on_board yes)
+		(dnp no)
+		(fields_autoplaced yes)
+		(property "Reference" "C9"
+			(at 86.36 85.0899 90)
+			(effects
+				(font
+					(size 1.524 1.524)
+				)
+				(justify left)
+			)
+		)
+		(property "Value" "33p"
+			(at 86.36 87.6299 90)
+			(effects
+				(font
+					(size 1.524 1.524)
+				)
+				(justify left)
+			)
+		)
+		(property "Footprint" "CAP_600F0R1AT250T_ATC"
+			(at 82.55 82.55 0)
+			(effects
+				(font
+					(size 1.27 1.27)
+					(italic yes)
+				)
+				(hide yes)
+			)
+		)
+		(property "Datasheet" "600F330FT250XT"
+			(at 82.55 82.55 0)
+			(effects
+				(font
+					(size 1.27 1.27)
+					(italic yes)
+				)
+				(hide yes)
+			)
+		)
+		(property "Description" "600F330FT250XT"
+			(at 82.55 82.55 0)
+			(effects
+				(font
+					(size 1.27 1.27)
+				)
+				(hide yes)
+			)
+		)
+		(pin "2"
+		)
+		(pin "1"
+		)
+		(instances
+			(project ""
+				(path "/fd6bac42-b74a-4329-b064-b676c79abc2c/4500e0af-ac1d-424f-9007-f4139dc7a85a"
+					(reference "C9")
+					(unit 1)
+				)
+			)
+		)
+	)
+	(symbol
 		(lib_id "power:GND")
 		(at 111.76 115.57 0)
@@
 	)
 	(symbol
+		(lib_id "RC0805FR_0751RL:RC0805FR-0751RL")
+		(at 71.12 80.01 180)
+		(unit 1)
+		(exclude_from_sim no)
+		(in_bom yes)
+		(on_board yes)
+		(dnp no)
+		(fields_autoplaced yes)
+		(property "Reference" "R9"
+			(at 64.77 73.66 0)
+			(effects
+				(font
+					(size 1.524 1.524)
+				)
+			)
+		)
+		(property "Value" "51"
+			(at 64.77 76.2 0)
+			(effects
+				(font
+					(size 1.524 1.524)
+				)
+			)
+		)
+		(property "Footprint" "RC0805N_YAG"
+			(at 71.12 80.01 0)
+			(effects
+				(font
+					(size 1.27 1.27)
+					(italic yes)
+				)
+				(hide yes)
+			)
+		)
+		(property "Datasheet" "RC0805FR-0751RL"
+			(at 71.12 80.01 0)
+			(effects
+				(font
+					(size 1.27 1.27)
+					(italic yes)
+				)
+				(hide yes)
+			)
+		)
+		(property "Description" "RC0805FR-0751RL"
+			(at 71.12 80.01 0)
+			(effects
+				(font
+					(size 1.27 1.27)
+				)
+				(hide yes)
+			)
+		)
+		(pin "1"
+		)
+		(pin "2"
+		)
+		(instances
+			(project ""
+				(path "/fd6bac42-b74a-4329-b064-b676c79abc2c/4500e0af-ac1d-424f-9007-f4139dc7a85a"
+					(reference "R9")
+					(unit 1)
+				)
+			)
+		)
+	)
+	(symbol
 		(lib_id "power:GND")
 		(at 100.33 87.63 270)
@@
 					(unit 1)
 				)
-			)
-		)
-	)
-	(symbol
-		(lib_id "Device:C")
-		(at 82.55 86.36 0)
-		(unit 1)
-		(exclude_from_sim no)
-		(in_bom yes)
-		(on_board yes)
-		(dnp no)
-		(fields_autoplaced yes)
-		(property "Reference" "C9"
-			(at 86.36 85.0899 0)
-			(effects
-				(font
-					(size 1.27 1.27)
-				)
-				(justify left)
-			)
-		)
-		(property "Value" "C"
-			(at 86.36 87.6299 0)
-			(effects
-				(font
-					(size 1.27 1.27)
-				)
-				(justify left)
-			)
-		)
-		(property "Footprint" "Resistor_SMD:R_0805_2012Metric_Pad1.20x1.40mm_HandSolder"
-			(at 83.5152 90.17 0)
-			(effects
-				(font
-					(size 1.27 1.27)
-				)
-				(hide yes)
-			)
-		)
-		(property "Datasheet" "~"
-			(at 82.55 86.36 0)
-			(effects
-				(font
-					(size 1.27 1.27)
-				)
-				(hide yes)
-			)
-		)
-		(property "Description" "Unpolarized capacitor"
-			(at 82.55 86.36 0)
-			(effects
-				(font
-					(size 1.27 1.27)
-				)
-				(hide yes)
-			)
-		)
-		(property "Part Number" ""
-			(at 82.55 86.36 0)
-			(effects
-				(font
-					(size 1.27 1.27)
-				)
-				(hide yes)
-			)
-		)
-		(pin "1"
-		)
-		(pin "2"
-		)
-		(instances
-			(project ""
-				(path "/fd6bac42-b74a-4329-b064-b676c79abc2c/4500e0af-ac1d-424f-9007-f4139dc7a85a"
-					(reference "C9")
-					(unit 1)
-				)
-			)
-		)
-	)
-	(symbol
-		(lib_id "Device:R")
-		(at 74.93 80.01 90)
-		(unit 1)
-		(exclude_from_sim no)
-		(in_bom yes)
-		(on_board yes)
-		(dnp no)
-		(fields_autoplaced yes)
-		(property "Reference" "R9"
-			(at 74.93 73.66 90)
-			(effects
-				(font
-					(size 1.27 1.27)
-				)
-			)
-		)
-		(property "Value" "R"
-			(at 74.93 76.2 90)
-			(effects
-				(font
-					(size 1.27 1.27)
-				)
-			)
-		)
-		(property "Footprint" "Resistor_SMD:R_0805_2012Metric_Pad1.20x1.40mm_HandSolder"
-			(at 74.93 81.788 90)
-			(effects
-				(font
-					(size 1.27 1.27)
-				)
-				(hide yes)
-			)
-		)
-		(property "Datasheet" "~"
-			(at 74.93 80.01 0)
-			(effects
-				(font
-					(size 1.27 1.27)
-				)
-				(hide yes)
-			)
-		)
-		(property "Description" "Resistor"
-			(at 74.93 80.01 0)
-			(effects
-				(font
-					(size 1.27 1.27)
-				)
-				(hide yes)
-			)
-		)
-		(property "Part Number" ""
-			(at 74.93 80.01 0)
-			(effects
-				(font
-					(size 1.27 1.27)
-				)
-				(hide yes)
-			)
-		)
-		(pin "1"
-		)
-		(pin "2"
-		)
-		(instances
-			(project ""
-				(path "/fd6bac42-b74a-4329-b064-b676c79abc2c/4500e0af-ac1d-424f-9007-f4139dc7a85a"
-					(reference "R9")
-					(unit 1)
-				)

Commit message: updated BOM
Parts:
- C9: Part Number (none) -> 600F330FT250XT
- D2, D7: Part Number (none) -> IR26-21C_L110_TR8
- D6: Part Number (none) -> US2AA
- R9: Part Number (none) -> RC0805FR-0751RL
- U3: Part Number (none) -> UCC5304DWVR
- U4: Part Number (none) -> TMV 0512SHI
Changed lines of the file:
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@@
+			)
+		)
+		(property "Part Number" "IR26-21C_L110_TR8"
+			(at 215.9 96.52 0)
+			(effects
+				(font
+					(size 1.27 1.27)
+				)
+				(hide yes)
 			)
 		)
@@
 			)
 		)
+		(property "Part Number" "600F330FT250XT"
+			(at 82.55 82.55 90)
+			(effects
+				(font
+					(size 1.27 1.27)
+				)
+				(hide yes)
+			)
+		)
 		(pin "2"
 		)
@@
 			)
 		)
+		(property "Part Number" "RC0805FR-0751RL"
+			(at 71.12 80.01 0)
+			(effects
+				(font
+					(size 1.27 1.27)
+				)
+				(hide yes)
+			)
+		)
 		(pin "1"
 		)
@@
 			)
 		)
+		(property "Part Number" "UCC5304DWVR"
+			(at 100.33 80.01 0)
+			(effects
+				(font
+					(size 1.27 1.27)
+				)
+				(hide yes)
+			)
+		)
 		(pin "8"
 		)
@@
 			)
 		)
+		(property "Part Number" "IR26-21C_L110_TR8"
+			(at 189.23 43.18 0)
+			(effects
+				(font
+					(size 1.27 1.27)
+				)
+				(hide yes)
+			)
+		)
 		(pin "1"
 		)
@@
 			)
 		)
+		(property "Part Number" "US2AA"
+			(at 182.88 82.55 0)
+			(effects
+				(font
+					(size 1.27 1.27)
+				)
+				(hide yes)
+			)
+		)
 		(pin "2"
 		)
@@
 			(at 93.98 52.07 0)
 			(effects
+				(font
+					(size 1.27 1.27)
+				)
+				(hide yes)
+			)
+		)
+		(property "Part Number" "TMV 0512SHI"
+			(at 93.98 52.07 0)
+			(effects
